Commit message: removed dependencies dae files not working

File: husky_description/urdf/accessories/kinect_camera.urdf.xacro (robot description, xacro)
@@ -34,5 +34,5 @@
         <origin xyz="0 0 0" rpy="0 0 ${M_PI/2}"/>
         <geometry>
-          <mesh filename="package://husky_description/meshes/accessories/kinect.dae" />
+          <mesh filename="/home/rigom/Desktop/Smile_Simulation/husky_description/meshes/accessories/kinect.dae" />
         </geometry>
       </visual>

File: husky_description/urdf/accessories/sensor_arch.urdf.xacro (robot description, xacro)
@@ -7,5 +7,5 @@
              <visual>
                  <geometry>
-                     <mesh filename="package://husky_description/meshes/accessories/${size}_mm_sensor_arch.dae" />
+                     <mesh filename="/home/rigom/Desktop/Smile_Simulation/husky_description/meshes/accessories/${size}_mm_sensor_arch.dae" />
                  </geometry>
              </visual>
@@ -13,5 +13,5 @@
                  <origin xyz="0 0 0" rpy="0 0 0"/>
                  <geometry>
-                     <mesh filename="package://husky_description/meshes/accessories/${size}_mm_sensor_arch.dae" />
+                     <mesh filename="/home/rigom/Desktop/Smile_Simulation/husky_description/meshes/accessories/${size}_mm_sensor_arch.dae" />
                  </geometry>
              </collision>

File: husky_description/urdf/accessories/sick_lms1xx_mount.urdf.xacro (robot description, xacro)
@@ -33,5 +33,5 @@
         <geometry>
           <!-- Origin of this mesh is the base of the bracket. -->
-          <mesh filename="package://husky_description/meshes/accessories/lms1xx_mount.dae" />
+          <mesh filename="/home/rigom/Desktop/Smile_Simulation/husky_description/meshes/accessories/lms1xx_mount.dae" />
         </geometry>
       </visual>

File: husky_description/urdf/decorations.urdf.xacro (robot description, xacro)
@@ -30,5 +30,5 @@
         <origin xyz="0 0 0" rpy="0 0 0" />
         <geometry>
-          <mesh filename="package://husky_description/meshes/top_chassis.dae" />
+          <mesh><uri>file:///home/rigom/Desktop/Smile_Simulation/husky_description/meshes/top_chassis.dae</uri></mesh>
         </geometry>
       </visual>
@@ -44,5 +44,5 @@
         <visual>
           <geometry>
-            <mesh filename="package://husky_description/meshes/user_rail.dae" />
+            <mesh><uri>file:///home/rigom/Desktop/Smile_Simulation/husky_description/meshes/user_rail.dae</uri></mesh>
           </geometry>
         </visual>
@@ -59,5 +59,5 @@
       <visual>
         <geometry>
-          <mesh filename="package://husky_description/meshes/bumper.dae" />
+          <mesh><uri>file:///home/rigom/Desktop/Smile_Simulation/husky_description/meshes/bumper.dae</uri></mesh>
         </geometry>
       </visual>
@@ -73,5 +73,5 @@
           <visual>
               <geometry>
-                  <mesh filename="package://husky_description/meshes/bumper_extension.dae" />
+                  <mesh><uri>file:///home/rigom/Desktop/Smile_Simulation/husky_description/meshes/bumper_extension.dae</uri></mesh>
               </geometry>
           </visual>
@@ -87,5 +87,5 @@
       <visual>
         <geometry>
-          <mesh filename="package://husky_description/meshes/bumper.dae" />
+          <mesh><uri>file:///home/rigom/Desktop/Smile_Simulation/husky_description/meshes/bumper.dae</uri></mesh>
         </geometry>
       </visual>
@@ -101,5 +101,5 @@
           <visual>
               <geometry>
-                  <mesh filename="package://husky_description/meshes/bumper_extension.dae" />
+                  <mesh><uri>file:///home/rigom/Desktop/Smile_Simulation/husky_description/meshes/bumper_extension.dae</uri></mesh>
               </geometry>
           </visual>
@@ -118,5 +118,5 @@
             <origin xyz="0 0 0" rpy="0 0 0" />
             <geometry>
-              <mesh filename="package://husky_description/meshes/large_top_plate.dae" />
+              <mesh><uri>file:///home/rigom/Desktop/Smile_Simulation/husky_description/meshes/large_top_plate.dae</uri></mesh>
             </geometry>
           </visual>
@@ -124,5 +124,5 @@
             <origin xyz="0 0 0" rpy="0 0 0"/>
             <geometry>
-              <mesh filename="package://husky_description/meshes/large_top_plate_collision.stl" />
+              <mesh><uri>file:///home/rigom/Desktop/Smile_Simulation/husky_description/meshes/large_top_plate_collision.stl</uri></mesh>
             </geometry>
           </collision>
@@ -152,5 +152,5 @@
             <origin xyz="0 0 0" rpy="0 0 0" />
             <geometry>
-              <mesh filename="package://husky_description/meshes/top_plate.dae" />
+              <mesh><uri>file:///home/rigom/Desktop/Smile_Simulation/husky_description/meshes/top_plate.dae</uri></mesh>
             </geometry>
           </visual>
@@ -158,5 +158,5 @@
             <origin xyz="0 0 0" rpy="0 0 0"/>
             <geometry>
-              <mesh filename="package://husky_description/meshes/top_plate.stl" />
+              <mesh><uri>file:///home/rigom/Desktop/Smile_Simulation/husky_description/meshes/top_plate.stl</uri></mesh>
             </geometry>
           </collision>

File: husky_description/urdf/husky.urdf.xacro (robot description, xacro)
@@ -1,29 +1,8 @@
 <?xml version="1.0"?>
-<!--
-Software License Agreement (BSD)
-\file      husky.urdf.xacro
-\authors   Paul Bovbel <pbovbel@clearpathrobotics.com>, Devon Ash <dash@clearpathrobotics.com>
-\copyright Copyright (c) 2015, Clearpath Robotics, Inc., All rights reserved.
-Redistribution and use in source and binary forms, with or without modification, are permitted provided that
-the following conditions are met:
- * Redistributions of source code must retain the above copyright notice, this list of conditions and the
-   following disclaimer.
- * Redistributions in binary form must reproduce the above copyright notice, this list of conditions and the
-   following disclaimer in the documentation and/or other materials provided with the distribution.
- * Neither the name of Clearpath Robotics nor the names of its contributors may be used to endorse or promote
-   products derived from this software without specific prior written permission.
-THIS SOFTWARE IS PROVIDED BY THE COPYRIGHT HOLDERS AND CONTRIBUTORS "AS IS" AND ANY EXPRESS OR IMPLIED WAR-
-RANTIES, INCLUDING, BUT NOT LIMITED TO, THE IMPLIED WARRANTIES OF MERCHANTABILITY AND FITNESS FOR A PARTICULAR
-PURPOSE ARE DISCLAIMED. IN NO EVENT SHALL THE COPYRIGHT HOLDER OR CONTRIBUTORS BE LIABLE FOR ANY DIRECT, IN-
-DIRECT, INCIDENTAL, SPECIAL, EXEMPLARY, OR CONSEQUENTIAL DAMAGES (INCLUDING, BUT NOT LIMITED TO, PROCUREMENT
-OF SUBSTITUTE GOODS OR SERVICES; LOSS OF USE, DATA, OR PROFITS; OR BUSINESS INTERRUPTION) HOWEVER CAUSED AND
-ON ANY THEORY OF LIABILITY, WHETHER IN CONTRACT, STRICT LIABILITY, OR TORT (INCLUDING NEGLIGENCE OR OTHERWISE)
-ARISING IN ANY WAY OUT OF THE USE OF THIS SOFTWARE, EVEN IF ADVISED OF THE POSSIBILITY OF SUCH DAMAGE.
--->
 <robot name="husky" xmlns:xacro="http://ros.org/wiki/xacro">
-  <xacro:arg name="laser_enabled" default="false" />
+  <xacro:arg name="laser_enabled" default="true" />
   <xacro:arg name="laser_xyz" default="$(optenv HUSKY_LMS1XX_XYZ 0.2206 0.0 0.00635)" />
   <xacro:arg name="laser_rpy" default="$(optenv HUSKY_LMS1XX_RPY 0.0 0.0 0.0)" />
-  <xacro:arg name="kinect_enabled" default="false" />
+  <xacro:arg name="kinect_enabled" default="true" />
   <xacro:arg name="kinect_xyz" default="$(optenv HUSKY_KINECT_XYZ 0 0 0)" />
   <xacro:arg name="kinect_rpy" default="$(optenv HUSKY_KINECT_RPY 0 0.18 3.14)" />
@@ -33,9 +12,9 @@
   <xacro:arg name="urdf_extras" default="empty.urdf" />
   <!-- Included URDF/XACRO Files -->
-  <xacro:include filename="$(find husky_description)/urdf/decorations.urdf.xacro" />
-  <xacro:include filename="$(find husky_description)/urdf/wheel.urdf.xacro" />
-  <xacro:include filename="$(find husky_description)/urdf/accessories/kinect_camera.urdf.xacro"/>
-  <xacro:include filename="$(find husky_description)/urdf/accessories/sick_lms1xx_mount.urdf.xacro"/>
-  <xacro:include filename="$(find husky_description)/urdf/accessories/sensor_arch.urdf.xacro"/>
+  <xacro:include filename="/home/rigom/Desktop/Smile_Simulation/husky_description/urdf/decorations.urdf.xacro" />
+  <xacro:include filename="/home/rigom/Desktop/Smile_Simulation/husky_description/urdf/wheel.urdf.xacro" />
+  <xacro:include filename="/home/rigom/Desktop/Smile_Simulation/husky_description/urdf/accessories/kinect_camera.urdf.xacro"/>
+  <xacro:include filename="/home/rigom/Desktop/Smile_Simulation/husky_description/urdf/accessories/sick_lms1xx_mount.urdf.xacro"/>
+  <xacro:include filename="/home/rigom/Desktop/Smile_Simulation/husky_description/urdf/accessories/sensor_arch.urdf.xacro"/>
   <xacro:property name="M_PI" value="3.14159"/>
   <!-- Base Size -->
@@ -55,5 +34,5 @@
       <origin xyz="0 0 0" rpy="0 0 0" />
       <geometry>
-        <mesh filename="package://husky_description/meshes/base_link.dae" />
+        <mesh><uri>file:///home/rigom/Desktop/Smile_Simulation/husky_description/meshes/base_link.dae</uri></mesh>
       </geometry>
     </visual>

File: husky_description/urdf/wheel.urdf.xacro (robot description, xacro)
@@ -32,5 +32,5 @@
 				<origin xyz="0 0 0" rpy="0 0 0" />
 				<geometry>
-					<mesh filename="package://husky_description/meshes/wheel.dae" />
+					<mesh><uri>file:///home/rigom/Desktop/Smile_Simulation/husky_description/meshes/wheel.dae</uri></mesh>
 				</geometry>
 			</visual>
